Commit message: debugging the simulation

File: motoman.urdf (robot description, URDF)
Before this commit: robot sda10f, 22 links, 21 joints
Links:
- link base_link: mass 0.00001 -> None

Commit message: fix rendering bug, add gitignore, python3 compatible

File: motoman.urdf (robot description, URDF)
Before this commit: robot sda10f, 22 links, 21 joints
Links:
- link arm_left_link_1_s: geometry collision mesh filename=sda10f_description/meshes/sda10f/collision/motoman_axis_s.s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; visual mesh filename=sda10f_description/meshes/sda10f/visual/motoman_axis_s.stl
- link arm_left_link_2_l: geometry collision mesh filename=sda10f_description/meshes/sda10f/collision/motoman_axis_l.s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; visual mesh filename=sda10f_description/meshes/sda10f/visual/motoman_axis_l.stl
- link arm_left_link_3_e: geometry collision mesh filename=sda10f_description/meshes/sda10f/collision/motoman_axis_e.s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; visual mesh filename=sda10f_description/meshes/sda10f/visual/motoman_axis_e.stl
- link arm_left_link_4_u: geometry collision mesh filename=sda10f_description/meshes/sda10f/collision/motoman_axis_u.s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; visual mesh filename=sda10f_description/meshes/sda10f/visual/motoman_axis_u.stl
- link arm_left_link_5_r: geometry collision mesh filename=sda10f_description/meshes/sda10f/collision/motoman_axis_r.s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; visual mesh filename=sda10f_description/meshes/sda10f/visual/motoman_axis_r.stl
- link arm_left_link_6_b: geometry collision mesh filename=sda10f_description/meshes/sda10f/collision/motoman_axis_b.s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; visual mesh filename=sda10f_description/meshes/sda10f/visual/motoman_axis_b.stl
- link arm_left_link_7_t: geometry collision mesh filename=sda10f_description/meshes/sda10f/collision/motoman_axis_t.s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; visual mesh filename=sda10f_description/meshes/sda10f/visual/motoman_axis_t.stl
- link arm_right_link_1_s: geometry collision mesh filename=sda10f_description/meshes/sda10f/collision/motoman_axis_s.s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; visual mesh filename=sda10f_description/meshes/sda10f/visual/motoman_axis_s.stl
- link arm_right_link_2_l: geometry collision mesh filename=sda10f_description/meshes/sda10f/collision/motoman_axis_l.s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; visual mesh filename=sda10f_description/meshes/sda10f/visual/motoman_axis_l.stl
- link arm_right_link_3_e: geometry collision mesh filename=sda10f_description/meshes/sda10f/collision/motoman_axis_e.s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; visual mesh filename=sda10f_description/meshes/sda10f/visual/motoman_axis_e.stl
- link arm_right_link_4_u: geometry collision mesh filename=sda10f_description/meshes/sda10f/collision/motoman_axis_u.s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; visual mesh filename=sda10f_description/meshes/sda10f/visual/motoman_axis_u.stl
- link arm_right_link_5_r: geometry collision mesh filename=sda10f_description/meshes/sda10f/collision/motoman_axis_r.s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; visual mesh filename=sda10f_description/meshes/sda10f/visual/motoman_axis_r.stl
- link arm_right_link_6_b: geometry collision mesh filename=sda10f_description/meshes/sda10f/collision/motoman_axis_b.s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; visual mesh filename=sda10f_description/meshes/sda10f/visual/motoman_axis_b.stl
- link arm_right_link_7_t: geometry collision mesh filename=sda10f_description/meshes/sda10f/collision/motoman_axis_t.s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; visual mesh filename=sda10f_description/meshes/sda10f/visual/motoman_axis_t.stl
- link base_link: geometry collision mesh filename=sda10f_description/meshes/sda10f/collision/motoman_base.stl; visual mesh filename=sda10f_description/meshes/sda10f/visual/motoman_base.stl
- link motoman_left_hand: geometry collision mesh filename=sda10f_description/meshes/sda10f/collision/baxter_suction2.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; visual mesh filename=sda10f_description/meshes/sda10f/visual/baxter_suction2.stl
- link motoman_right_hand: geometry collision mesh filename=sda10f_description/meshes/sda10f/collision/modelO42.stl; visual mesh filename=sda10f_description/meshes/sda10f/visual/modelO42.stl
- link torso_link: geometry collision mesh filename=sda10f_description/meshes/sda10f/collision/motoman_axis_b1.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; visual mesh filename=sda10f_description/meshes/sda10f/visual/motoman_axis_b1.stl
