Commit message: wrap the directory into ROS workspace

File: src/pybullet_motoman/src/motoman.urdf (robot description, URDF)
Before this commit: robot sda10f, 22 links, 21 joints
Links:
- link motoman_left_hand: geometry collision mesh filename=sda10f_description/meshes/sda10f/collision/vacuum_gripper_n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; visual mesh filename=sda10f_description/meshes/sda10f/visual/vacuum_gripper_no_m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
