Commit message: Change urdf for Robotiq gripper

File: urdf/motoman.urdf (robot description, URDF)
Before this commit: robot sda10f, 22 links, 21 joints
Links:
- removed link motoman_right_hand
- added link left_inner_finger; collision mesh filename=package://pybullet_motoman/urdf/robotiq_85/collision/roboti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 scale=0.001 0.001 0.001; visual mesh filename=package://pybullet_motoman/urdf/robotiq_85/visual/robotiq_a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 scale=0.001 0.001 0.001
- added link left_inner_finger_pad; collision box size=0.022 0.00635 0.0375; visual box size=0.022 0.00635 0.0375
- added link left_inner_knuckle; collision mesh filename=package://pybullet_motoman/urdf/robotiq_85/collision/roboti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 scale=0.001 0.001 0.001; visual mesh filename=package://pybullet_motoman/urdf/robotiq_85/visual/robotiq_a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 scale=0.001 0.001 0.001
- added link left_outer_finger; collision mesh filename=package://pybullet_motoman/urdf/robotiq_85/collision/roboti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 scale=0.001 0.001 0.001; visual mesh filename=package://pybullet_motoman/urdf/robotiq_85/visual/robotiq_a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 scale=0.001 0.001 0.001
- added link left_outer_knuckle; collision mesh filename=package://pybullet_motoman/urdf/robotiq_85/collision/roboti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 scale=0.001 0.001 0.001; visual mesh filename=package://pybullet_motoman/urdf/robotiq_85/visual/robotiq_a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 scale=0.001 0.001 0.001
- added link right_inner_finger; collision mesh filename=package://pybullet_motoman/urdf/robotiq_85/collision/roboti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 scale=0.001 0.001 0.001; visual mesh filename=package://pybullet_motoman/urdf/robotiq_85/visual/robotiq_a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 scale=0.001 0.001 0.001
- added link right_inner_finger_pad; collision box size=0.022 0.00635 0.0375; visual box size=0.022 0.00635 0.0375
- added link right_inner_knuckle; collision mesh filename=package://pybullet_motoman/urdf/robotiq_85/collision/roboti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 scale=0.001 0.001 0.001; visual mesh filename=package://pybullet_motoman/urdf/robotiq_85/visual/robotiq_a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 scale=0.001 0.001 0.001
- added link right_outer_finger; collision mesh filename=package://pybullet_motoman/urdf/robotiq_85/collision/roboti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 scale=0.001 0.001 0.001; visual mesh filename=package://pybullet_motoman/urdf/robotiq_85/visual/robotiq_a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 scale=0.001 0.001 0.001
- added link right_outer_knuckle; collision mesh filename=package://pybullet_motoman/urdf/robotiq_85/collision/roboti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 scale=0.001 0.001 0.001; visual mesh filename=package://pybullet_motoman/urdf/robotiq_85/visual/robotiq_a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 scale=0.001 0.001 0.001
- added link robotiq_arg2f_base_link, mass 0.22652; collision mesh filename=package://pybullet_motoman/urdf/robotiq_85/collision/roboti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; visual mesh filename=package://pybullet_motoman/urdf/robotiq_85/visual/robotiq_a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 scale=0.001 0.001 0.001
Joints:
- added joint finger_joint: type revolute, parent robotiq_arg2f_base_link, child left_outer_knuckle, origin xyz=0 -0.0306011 0.054904 rpy=0 0 3.14159265359, axis 1 0 0, limit lower=0 upper=0.8 effort=1000 velocity=2.0
- added joint left_inner_finger_joint: type revolute, parent left_outer_finger, child left_inner_finger, origin xyz=0 0.0061 0.0471 rpy=0 0 0, axis 1 0 0, limit lower=-0.8757 upper=0 effort=1000 velocity=2.0, mimic joint=finger_joint multiplier=-1 offset=0
- added joint left_inner_finger_pad_joint: type fixed, parent left_inner_finger, child left_inner_finger_pad, origin xyz=0 -0.0220203446692936 0.03242 rpy=0 0 0, axis 0 0 1
- added joint left_inner_knuckle_joint: type revolute, parent robotiq_arg2f_base_link, child left_inner_knuckle, origin xyz=0 -0.0127 0.06142 rpy=0 0 3.14159265359, axis 1 0 0, limit lower=0 upper=0.8757 effort=1000 velocity=2.0, mimic joint=finger_joint multiplier=1 offset=0
- added joint left_outer_finger_joint: type fixed, parent left_outer_knuckle, child left_outer_finger, origin xyz=0 0.0315 -0.0041 rpy=0 0 0, axis 1 0 0
- added joint right_inner_finger_joint: type revolute, parent right_outer_finger, child right_inner_finger, origin xyz=0 0.0061 0.0471 rpy=0 0 0, axis 1 0 0, limit lower=-0.8757 upper=0 effort=1000 velocity=2.0, mimic joint=finger_joint multiplier=-1 offset=0
- added joint right_inner_finger_pad_joint: type fixed, parent right_inner_finger, child right_inner_finger_pad, origin xyz=0 -0.0220203446692936 0.03242 rpy=0 0 0, axis 0 0 1
- added joint right_inner_knuckle_joint: type revolute, parent robotiq_arg2f_base_link, child right_inner_knuckle, origin xyz=0 0.0127 0.06142 rpy=0 0 0.0, axis 1 0 0, limit lower=0 upper=0.8757 effort=1000 velocity=2.0, mimic joint=finger_joint multiplier=1 offset=0
- added joint right_outer_finger_joint: type fixed, parent right_outer_knuckle, child right_outer_finger, origin xyz=0 0.0315 -0.0041 rpy=0 0 0, axis 1 0 0
- added joint right_outer_knuckle_joint: type revolute, parent robotiq_arg2f_base_link, child right_outer_knuckle, origin xyz=0 0.0306011 0.054904 rpy=0 0 0, axis 1 0 0, limit lower=0 upper=0.81 effort=1000 velocity=2.0, mimic joint=finger_joint multiplier=1 offset=0
- joint motoman_left_joint_pre_ee: origin xyz=0 0 0.0 rpy=3.141 0 0 -> xyz=0 0 0.0 rpy=3.1416 0 0
- joint motoman_right_joint_ee: origin xyz=0 0.03 0.18 rpy=0 0 0 -> xyz=0 0 0.135 rpy=0 0 0; parent motoman_right_hand -> robotiq_arg2f_base_link
- joint motoman_right_joint_pre_ee: child motoman_right_hand -> robotiq_arg2f_base_link; origin xyz=0 0 0.0 rpy=3.141 0 0 -> xyz=0 0 0.0 rpy=3.1416 0 0

Commit message: improved planning and has been tested

File: urdf/motoman.urdf (robot description, URDF)
Before this commit: robot sda10f, 32 links, 31 joints
Joints:
- joint arm_left_joint_tool0: origin xyz=0 0 -0.0325 rpy=0 0 -3.13 -> xyz=0 0 -0.025 rpy=0 0 -3.13
- joint arm_right_joint_tool0: origin xyz=0 0 -0.0325 rpy=0 0 -3.13 -> xyz=0 0 -0.025 rpy=0 0 -3.13

Commit message: (1) better planning (2) fix robotiq gripper issue (3) add more motion type (4) better drop the object

File: urdf/motoman.urdf (robot description, URDF)
Before this commit: robot sda10f, 32 links, 31 joints
Joints:
- joint arm_left_joint_4_u: limit lower=-2.36 upper=2.36 effort=0 velocity=2.95 -> lower=-2.36 upper=0 effort=0 velocity=2.95
- joint arm_right_joint_4_u: limit lower=-2.36 upper=2.36 effort=0 velocity=2.95 -> lower=-2.36 upper=0 effort=0 velocity=2.95

Commit message: tune parameter to match real + change reset planning

File: urdf/motoman.urdf (robot description, URDF)
Before this commit: robot sda10f, 32 links, 31 joints
Joints:
- joint arm_left_joint_tool0: origin xyz=0 0 -0.025 rpy=0 0 -3.13 -> xyz=0 0 -0.09 rpy=0 0 -3.13
- joint motoman_right_joint_pre_ee: origin xyz=0 0 0.0 rpy=3.1416 0 0 -> xyz=0 0 0.0 rpy=3.1416 0 1.57

Commit message: apply sim2real parameter tuning in execution node

File: urdf/motoman.urdf (robot description, URDF)
Before this commit: robot sda10f, 32 links, 31 joints
Joints:
- joint arm_left_joint_2_l: limit lower=-1.90 upper=1.90 effort=0 velocity=2.95 -> lower=-1.90 upper=1.70 effort=0 velocity=2.95
- joint arm_right_joint_2_l: limit lower=-1.90 upper=1.90 effort=0 velocity=2.95 -> lower=-1.90 upper=1.70 effort=0 velocity=2.95

Commit message: add approachToPlacement functionality

File: urdf/motoman.urdf (robot description, URDF)
Before this commit: robot sda10f, 32 links, 31 joints
Links:
- removed link torso_link
- added link torso_link_b1; collision mesh filename=package://pybullet_motoman/urdf/sda10f_description/meshes/s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; visual mesh filename=package://pybullet_motoman/urdf/sda10f_description/meshes/s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
Joints:
- removed joint torso_joint_0
- added joint torso_joint_b1: type fixed, parent base_link, child torso_link_b1, origin xyz=0.09257 0 0.877 rpy=0 0 0
- joint arm_left_joint_1_s: parent torso_link -> torso_link_b1
- joint arm_left_joint_2_l: limit lower=-1.90 upper=1.70 effort=0 velocity=2.95 -> lower=-1.90 upper=1.90 effort=0 velocity=2.95
- joint arm_left_joint_4_u: limit lower=-2.36 upper=0 effort=0 velocity=2.95 -> lower=-2.36 upper=2.36 effort=0 velocity=2.95
- joint arm_right_joint_1_s: parent torso_link -> torso_link_b1
- joint arm_right_joint_2_l: limit lower=-1.90 upper=1.70 effort=0 velocity=2.95 -> lower=-1.90 upper=1.90 effort=0 velocity=2.95
- joint arm_right_joint_4_u: limit lower=-2.36 upper=0 effort=0 velocity=2.95 -> lower=-2.36 upper=2.36 effort=0 velocity=2.95

Commit message: fix the goal connection and add moveit trajectory execution

File: urdf/motoman.urdf (robot description, URDF)
Before this commit: robot sda10f, 32 links, 31 joints
Joints:
- joint torso_joint_b1: axis (none) -> 0 0 1; limit (none) -> lower=-2.9570 upper=2.9570 effort=100 velocity=2.26; type fixed -> revolute
